File: Fight Stick 2/Untitled/Untitled.kicad_pcb (KiCad board)
At the start: 2 copper layers, 146.2 x 62.1 mm, 18 parts, among them U1 Elite-C

Commit message: second version upload
Parts:
- removed U1: Elite-C, Keebio-Parts.pretty-master:Elite-C-castellated-24pin-holes
- added H4: MountingHole, MountingHole:MountingHole_2.2mm_M2_DIN965_Pad, F.Cu at (78.4, 74.2)
- added U2: ProMicro, PCM_marbastlib-xp-promicroish:ProMicro_USBdn, F.Cu at (96.8, 74.2)
- MX1, MX10, MX11, MX12, MX13, MX14, MX2, MX3, MX4, MX5, MX6, MX7, MX8, MX9: footprint keyswitches.pretty-2.1:Kailh_socket_MX_optional -> Fight Stick 2:MX_optional
- renumbered H4 to H3
Routing:
- net MX2: track 30.2 -> 55.4 mm
- net MX1: track 52.3 -> 31.3 mm
- net MX7: track 129.4 -> 144.4 mm, vias 0 -> 2
- net MX6: track 108.8 -> 118.2 mm
- net MX5: track 88.0 -> 95.8 mm
- net MX3: track 46.2 -> 53.1 mm
- net MX4: track 65.5 -> 72.0 mm
- net MX11: track 85.6 -> 80.4 mm
- net MX10: track 72.9 -> 68.7 mm
- net MX9: track 45.9 -> 44.1 mm
- net MX8: track 30.3 -> 28.5 mm
- net MX12: track 102.5 -> 101.4 mm
- net MX14: track 133.5 -> 133.0 mm
- net GND: vias 25 -> 69
