File: FightStickMini.HighProfile/Kicad Files/Untitled.kicad_pcb (KiCad board)
At the start: 2 copper layers, 146.2 x 62.1 mm, 19 parts, among them U2 ProMicro

Commit message: lowprofile
Routing:
- net GND: vias 69 -> 46
Other:
- board text added: "FighterMini.V2.HighProfile.ProMicro.GP2040.Mega32U4."
- board text added: "PM20.GP28.MX12.MK.PS(Tri).X(Y) PM18.GP26.MX6.HP.PS(L1).X(LB) PM19.GP27.MX13.HK.PS(R1).X(RB) PM2.GP2.MX7.TP.PS(L2).X(LT) PM3.GP3.MX14.TK.PS(R2).X(RT) PM8.GP8.MX8.S1.PS(Sel).X(Bac) PM7.GP7.MX9.S2.PS(Sta).X(Sta)"
- board text added: "PM6.GP6.MX10.UP.PS.UP.XX PM14.GP20.MX2.DOWN.PS.DOW.XX PM16.GP23.MX1.LEFT.PS.LEF.XX PM15.GP22.MX3.RIGHT.PS.RIG.XX PM21.GP29.MX4.LP.PS(Squ).X(X) PM5.GP5.MX11.LK.PS(X).X(A) PM4.GP4.MX5.MP.PS(Cir).X(B)"
- board text removed: "FIGHTER MINI V2 PRO MICRO"
Changed lines of the file:
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@@
   (gr_arc (start 221.174256 102.026735) (mid 220.295561 104.148017) (end 218.174256 105.026735)
     (stroke (width 0.1) (type default)) (layer "Edge.Cuts"))
-  (gr_text "FIGHTER MINI V2 PRO MICRO\n" (at 189.738 100.838) (layer "B.SilkS")
+  (gr_text "PM20.GP28.MX12.MK.PS(Tri).X(Y)\nPM18.GP26.MX6.HP.PS(L1).X(LB)\nPM19.GP27.MX13.HK.PS(R1).X(RB)\nPM2.GP2.MX7.TP.PS(L2).X(LT)\nPM3.GP3.MX14.TK.PS(R2).X(RT)\nPM8.GP8.MX8.S1.PS(Sel).X(Bac)\nPM7.GP7.MX9.S2.PS(Sta).X(Sta)" (at 183.769 100.711) (layer "B.SilkS")
+    (effects (font (size 1 1) (thickness 0.15)) (justify left bottom mirror))
+  )
+  (gr_text "PM6.GP6.MX10.UP.PS.UP.XX\nPM14.GP20.MX2.DOWN.PS.DOW.XX\nPM16.GP23.MX1.LEFT.PS.LEF.XX\nPM15.GP22.MX3.RIGHT.PS.RIG.XX\nPM21.GP29.MX4.LP.PS(Squ).X(X)\nPM5.GP5.MX11.LK.PS(X).X(A)\nPM4.GP4.MX5.MP.PS(Cir).X(B)" (at 210.693 100.711) (layer "B.SilkS")
+    (effects (font (size 1 1) (thickness 0.15)) (justify left bottom mirror))
+  )
+  (gr_text "FighterMini.V2.HighProfile.ProMicro.GP2040.Mega32U4." (at 210.566 103.378) (layer "B.SilkS")
     (effects (font (size 1 1) (thickness 0.15)) (justify left bottom mirror))
   )
@@
   (via (at 185.166 85.598) (size 0.8) (drill 0.4) (layers "F.Cu" "B.Cu") (free) (net 2))
   (via (at 95.504 46.101) (size 0.8) (drill 0.4) (layers "F.Cu" "B.Cu") (free) (net 2))
-  (via (at 210.327 102.997) (size 0.8) (drill 0.4) (layers "F.Cu" "B.Cu") (free) (net 2))
-  (via (at 158.877 102.997) (size 0.8) (drill 0.4) (layers "F.Cu" "B.Cu") (free) (net 2))
   (via (at 181.483 52.324) (size 0.8) (drill 0.4) (layers "F.Cu" "B.Cu") (free) (net 2))
-  (via (at 177.927 91.567) (size 0.8) (drill 0.4) (layers "F.Cu" "B.Cu") (free) (net 2))
+  (via (at 185.166 99.568) (size 0.8) (drill 0.4) (layers "F.Cu" "B.Cu") (free) (net 2))
   (via (at 141.0208 51.308) (size 0.8) (drill 0.4) (layers "F.Cu" "B.Cu") (free) (net 2))
   (via (at 95.504 102.235) (size 0.8) (drill 0.4) (layers "F.Cu" "B.Cu") (free) (net 2))
@@
   (via (at 184.15 45) (size 0.8) (drill 0.4) (layers "F.Cu" "B.Cu") (free) (net 2))
   (via (at 152.527 96.774) (size 0.8) (drill 0.4) (layers "F.Cu" "B.Cu") (free) (net 2))
-  (via (at 165.227 91.567) (size 0.8) (drill 0.4) (layers "F.Cu" "B.Cu") (free) (net 2))
   (via (at 116 103) (size 0.8) (drill 0.4) (layers "F.Cu" "B.Cu") (free) (net 2))
   (via (at 146.177 102.997) (size 0.8) (drill 0.4) (layers "F.Cu" "B.Cu") (free) (net 2))
-  (via (at 190.627 102.997) (size 0.8) (drill 0.4) (layers "F.Cu" "B.Cu") (free) (net 2))
+  (via (at 212.598 100.203) (size 0.8) (drill 0.4) (layers "F.Cu" "B.Cu") (free) (net 2))
   (via (at 146.177 91.567) (size 0.8) (drill 0.4) (layers "F.Cu" "B.Cu") (free) (net 2))
-  (via (at 203.327 91.567) (size 0.8) (drill 0.4) (layers "F.Cu" "B.Cu") (free) (net 2))
   (via (at 190.5 45) (size 0.8) (drill 0.4) (layers "F.Cu" "B.Cu") (free) (net 2))
-  (via (at 197.327 96.774) (size 0.8) (drill 0.4) (layers "F.Cu" "B.Cu") (free) (net 2))
-  (via (at 184.277 91.567) (size 0.8) (drill 0.4) (layers "F.Cu" "B.Cu") (free) (net 2))
-  (via (at 203.327 102.997) (size 0.8) (drill 0.4) (layers "F.Cu" "B.Cu") (free) (net 2))
-  (via (at 158.877 91.567) (size 0.8) (drill 0.4) (layers "F.Cu" "B.Cu") (free) (net 2))
+  (via (at 212.217 91.567) (size 0.8) (drill 0.4) (layers "F.Cu" "B.Cu") (free) (net 2))
   (via (at 141.605 77.597) (size 0.8) (drill 0.4) (layers "F.Cu" "B.Cu") (free) (net 2))
   (via (at 141 45) (size 0.8) (drill 0.4) (layers "F.Cu" "B.Cu") (free) (net 2))
-  (via (at 197.327 91.567) (size 0.8) (drill 0.4) (layers "F.Cu" "B.Cu") (free) (net 2))
-  (via (at 171.577 91.567) (size 0.8) (drill 0.4) (layers "F.Cu" "B.Cu") (free) (net 2))
   (via (at 116.586 82.296) (size 0.8) (drill 0.4) (layers "F.Cu" "B.Cu") (free) (net 2))
   (via (at 129.286 82.423) (size 0.8) (drill 0.4) (layers "F.Cu" "B.Cu") (free) (net 2))
-  (via (at 165.227 102.997) (size 0.8) (drill 0.4) (layers "F.Cu" "B.Cu") (free) (net 2))
   (via (at 136.0208 51.308) (size 0.8) (drill 0.4) (layers "F.Cu" "B.Cu") (free) (net 2))
   (via (at 200.533 73.279) (size 0.8) (drill 0.4) (layers "F.Cu" "B.Cu") (free) (net 2))
-  (via (at 165.227 96.774) (size 0.8) (drill 0.4) (layers "F.Cu" "B.Cu") (free) (net 2))
   (via (at 89.281 74.295) (size 0.8) (drill 0.4) (layers "F.Cu" "B.Cu") (free) (net 2))
   (via (at 118.999 87.757) (size 0.8) (drill 0.4) (layers "F.Cu" "B.Cu") (free) (net 2))
@@
   (via (at 162.56 51.181) (size 0.8) (drill 0.4) (layers "F.Cu" "B.Cu") (free) (net 2))
   (via (at 196.85 45) (size 0.8) (drill 0.4) (layers "F.Cu" "B.Cu") (free) (net 2))
-  (via (at 184.277 102.997) (size 0.8) (drill 0.4) (layers "F.Cu" "B.Cu") (free) (net 2))
-  (via (at 190.627 91.567) (size 0.8) (drill 0.4) (layers "F.Cu" "B.Cu") (free) (net 2))
   (via (at 136.0208 58.5724) (size 0.8) (drill 0.4) (layers "F.Cu" "B.Cu") (free) (net 2))
-  (via (at 171.577 96.774) (size 0.8) (drill 0.4) (layers "F.Cu" "B.Cu") (free) (net 2))
   (via (at 152.527 102.997) (size 0.8) (drill 0.4) (layers "F.Cu" "B.Cu") (free) (net 2))
   (via (at 165.354 84.074) (size 0.8) (drill 0.4) (layers "F.Cu" "B.Cu") (free) (net 2))
-  (via (at 177.927 102.997) (size 0.8) (drill 0.4) (layers "F.Cu" "B.Cu") (free) (net 2))
-  (via (at 190.627 96.774) (size 0.8) (drill 0.4) (layers "F.Cu" "B.Cu") (free) (net 2))
-  (via (at 171.577 102.997) (size 0.8) (drill 0.4) (layers "F.Cu" "B.Cu") (free) (net 2))
   (via (at 203 45) (size 0.8) (drill 0.4) (layers "F.Cu" "B.Cu") (free) (net 2))
-  (via (at 210.327 91.567) (size 0.8) (drill 0.4) (layers "F.Cu" "B.Cu") (free) (net 2))
   (via (at 116.84 66.802) (size 0.8) (drill 0.4) (layers "F.Cu" "B.Cu") (free) (net 2))
   (via (at 216.535 91.567) (size 0.8) (drill 0.4) (layers "F.Cu" "B.Cu") (free) (net 2))
-  (via (at 210.327 96.774) (size 0.8) (drill 0.4) (layers "F.Cu" "B.Cu") (free) (net 2))
-  (via (at 197.327 102.997) (size 0.8) (drill 0.4) (layers "F.Cu" "B.Cu") (free) (net 2))
   (via (at 136 45) (size 0.8) (drill 0.4) (layers "F.Cu" "B.Cu") (free) (net 2))
   (via (at 82.677 76.708) (size 0.8) (drill 0.4) (layers "F.Cu" "B.Cu") (free) (net 2))
+  (via (at 160.909 102.997) (size 0.8) (drill 0.4) (layers "F.Cu" "B.Cu") (free) (net 2))
   (via (at 152.527 91.567) (size 0.8) (drill 0.4) (layers "F.Cu" "B.Cu") (free) (net 2))
   (via (at 218.186 69.596) (size 0.8) (drill 0.4) (layers "F.Cu" "B.Cu") (free) (net 2))
   (via (at 210 49) (size 0.8) (drill 0.4) (layers "F.Cu" "B.Cu") (free) (net 2))
   (via (at 122 103) (size 0.8) (drill 0.4) (layers "F.Cu" "B.Cu") (free) (net 2))
-  (via (at 184.277 96.774) (size 0.8) (drill 0.4) (layers "F.Cu" "B.Cu") (free) (net 2))
   (via (at 114.554 46.228) (size 0.8) (drill 0.4) (layers "F.Cu" "B.Cu") (free) (net 2))
   (via (at 133.096 66.802) (size 0.8) (drill 0.4) (layers "F.Cu" "B.Cu") (free) (net 2))
-  (via (at 158.877 96.774) (size 0.8) (drill 0.4) (layers "F.Cu" "B.Cu") (free) (net 2))
   (via (at 210 45) (size 0.8) (drill 0.4) (layers "F.Cu" "B.Cu") (free) (net 2))
   (via (at 200.66 55.118) (size 0.8) (drill 0.4) (layers "F.Cu" "B.Cu") (free) (net 2))
-  (via (at 177.927 96.774) (size 0.8) (drill 0.4) (layers "F.Cu" "B.Cu") (free) (net 2))
-  (via (at 203.327 96.774) (size 0.8) (drill 0.4) (layers "F.Cu" "B.Cu") (free) (net 2))
   (segment (start 87.884 63.754) (end 89.408 62.23) (width 0.25) (layer "F.Cu") (net 3))
   (segment (start 96.266 51.562) (end 99.314 48.514) (width 0.25) (layer "F.Cu") (net 3))
