File: FightStickMini.LowProfile/Kicad Files/Untitled.kicad_sch (KiCad schematic)
At the start: 19 parts, among them U2 ProMicro

Commit message: update
Parts:
- added S1: MX_stab, PCM_marbastlib-mx:STAB_MX_P_6.25u, symbol marbastlib-mx:MX_stab
- U2: footprint Fight Stick 2:ProMicro_USBdn -> PCM_marbastlib-xp-promicroish:Elite-C_ACH
Changed lines of the file:
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@@
+    )
+  )
+  (symbol (lib_id "marbastlib-mx:MX_stab") (at 156.21 91.44 0) (unit 1)
+    (in_bom yes) (on_board yes) (dnp no) (fields_autoplaced)
+    (property "Reference" "S1" (at 162.56 90.043 0)
+      (effects (font (size 1.27 1.27)) (justify left))
+    )
+    (property "Value" "MX_stab" (at 162.56 92.583 0)
+      (effects (font (size 1.27 1.27)) (justify left))
+    )
+    (property "Footprint" "PCM_marbastlib-mx:STAB_MX_P_6.25u" (at 156.21 91.44 0)
+      (effects (font (size 1.27 1.27)) hide)
+    )
+    (property "Datasheet" "" (at 156.21 91.44 0)
+      (effects (font (size 1.27 1.27)) hide)
+    )
+    (instances
+      (project "Untitled"
+        (path "/9b1b67d5-31e7-4504-9acf-822c869dae16"
+          (reference "S1") (unit 1)
+        )
+      )
     )
   )
@@
       (effects (font (size 1.27 1.27)))
     )
-    (property "Footprint" "Fight Stick 2:ProMicro_USBdn" (at 71.12 85.09 0)
-      (effects (font (size 1.27 1.27)) hide)
-    )
+    (property "Footprint" "PCM_marbastlib-xp-promicroish:Elite-C_ACH" (at 71.12 85.09 0)
+      (effects (font (size 1.27 1.27)) hide)
+    )
